File: rotor.kicad_pcb (KiCad board)
At the start: 2 copper layers, 15.5 x 33.6 mm, 27 parts, among them J1 INPUT, J2 Motor, U1 STSPIN220/STSPIN250

Commit message: add readme
Parts:
- C1, C2: value C -> 1uF
- C3: value C -> 12nF
- R10: value R -> 1KΩ
- R12: value R -> 47KΩ
- R14, R15: value 0.3Ω -> Rsense
- R4, R5: value R -> Rref
- R7: value R -> 10KΩ
Routing:
- net Net-(U1-TOFF): track 11.2 -> 9.16 mm
- net GND: track 20.4 -> 21.7 mm, vias 14 -> 13
Changed lines of the file:
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@@
         (effects (font (size 1 1) (thickness 0.15)))
     )
-    (fp_text value "C" (at 0 1.43) (layer "F.Fab")
+    (fp_text value "1uF" (at 0 1.43) (layer "F.Fab")
         (effects (font (size 1 1) (thickness 0.15)))
     )
@@
         (effects (font (size 1 1) (thickness 0.15)))
     )
-    (fp_text value "R" (at 0 1.43) (layer "F.Fab")
+    (fp_text value "47KΩ" (at 0 1.43) (layer "F.Fab")
         (effects (font (size 1 1) (thickness 0.15)))
     )
@@
         (effects (font (size 1 1) (thickness 0.15)))
     )
-    (fp_text value "R" (at 0 1.43) (layer "F.Fab")
+    (fp_text value "Rref" (at 0 1.43) (layer "F.Fab")
         (effects (font (size 1 1) (thickness 0.15)))
     )
@@
         (effects (font (size 1 1) (thickness 0.15)))
     )
-    (fp_text value "C" (at 0 1.43) (layer "F.Fab")
+    (fp_text value "12nF" (at 0 1.43) (layer "F.Fab")
         (effects (font (size 1 1) (thickness 0.15)))
     )
@@
         (effects (font (size 1 1) (thickness 0.15)))
     )
-    (fp_text value "0.3Ω" (at 0 1.82 90) (layer "F.Fab")
+    (fp_text value "Rsense" (at 0 1.82 90) (layer "F.Fab")
         (effects (font (size 1 1) (thickness 0.15)))
     )
@@
         (effects (font (size 1 1) (thickness 0.15)))
     )
-    (fp_text value "R" (at 0 1.43) (layer "F.Fab")
+    (fp_text value "1KΩ" (at 0 1.43) (layer "F.Fab")
         (effects (font (size 1 1) (thickness 0.15)))
     )
@@
         (effects (font (size 1 1) (thickness 0.15)))
     )
-    (fp_text value "R" (at 0 1.43) (layer "F.Fab")
+    (fp_text value "10KΩ" (at 0 1.43) (layer "F.Fab")
         (effects (font (size 1 1) (thickness 0.15)))
     )
@@
         (effects (font (size 1 1) (thickness 0.15)))
     )
-    (fp_text value "0.3Ω" (at 0 1.82 90) (layer "F.Fab")
+    (fp_text value "Rsense" (at 0 1.82 90) (layer "F.Fab")
         (effects (font (size 1 1) (thickness 0.15)))
     )
@@
         (effects (font (size 1 1) (thickness 0.15)))
     )
-    (fp_text value "R" (at 0 1.43) (layer "F.Fab")
+    (fp_text value "Rref" (at 0 1.43) (layer "F.Fab")
         (effects (font (size 1 1) (thickness 0.15)))
     )
@@
         (effects (font (size 1 1) (thickness 0.15)))
     )
-    (fp_text value "C" (at 0 1.43) (layer "F.Fab")
+    (fp_text value "1uF" (at 0 1.43) (layer "F.Fab")
         (effects (font (size 1 1) (thickness 0.15)))
     )
@@
   (segment (start 109.157 50.03) (end 109.157 49.775707) (width 0.3) (layer "F.Cu") (net 1))
   (segment (start 108.976817 53.594) (end 109.157 53.594) (width 0.3) (layer "F.Cu") (net 1))
+  (segment (start 104.3432 50.0002) (end 104.381 50.038) (width 0.3) (layer "F.Cu") (net 1))
+  (segment (start 104.3432 49.8856) (end 104.3432 50.0002) (width 0.3) (layer "F.Cu") (net 1))
   (segment (start 107.045553 43.558553) (end 106.667 43.18) (width 0.3) (layer "F.Cu") (net 1))
   (segment (start 105.931 55.372) (end 106.934 55.372) (width 0.3) (layer "F.Cu") (net 1))
-  (segment (start 104.4448 50.038) (end 105.156 49.3268) (width 0.3) (layer "F.Cu") (net 1))
   (segment (start 109.157 51.816) (end 108.817507 51.816) (width 0.3) (layer "F.Cu") (net 1))
   (segment (start 109.010553 49.422153) (end 108.712 49.1236) (width 0.3) (layer "F.Cu") (net 1))
@@
   (segment (start 102.679 49.547107) (end 102.679 50.038) (width 0.3) (layer "F.Cu") (net 1))
   (segment (start 101.029 55.372) (end 101.029 55.689) (width 0.3) (layer "F.Cu") (net 1))
+  (segment (start 104.381 50.038) (end 104.381 49.3285) (width 0.3) (layer "F.Cu") (net 1))
   (segment (start 102.629 53.594) (end 102.629 53.179107) (width 0.3) (layer "F.Cu") (net 1))
   (segment (start 108.463953 51.669553) (end 108.2548 51.4604) (width 0.3) (layer "F.Cu") (net 1))
+  (segment (start 104.381 49.3285) (end 103.378 48.3255) (width 0.3) (layer "F.Cu") (net 1))
   (segment (start 102.482553 52.825553) (end 102.362 52.705) (width 0.3) (layer "F.Cu") (net 1))
   (segment (start 106.520553 40.502553) (end 105.642 39.624) (width 0.3) (layer "F.Cu") (net 1))
@@
   (segment (start 106.667 43.18) (end 106.667 40.856107) (width 0.3) (layer "F.Cu") (net 1))
   (segment (start 107.192 45.2485) (end 107.192 46.278893) (width 0.3) (layer "F.Cu") (net 1))
-  (segment (start 104.381 50.038) (end 104.4448 50.038) (width 0.3) (layer "F.Cu") (net 1))
   (segment (start 103.378 48.3255) (end 103.378 48.433893) (width 0.3) (layer "F.Cu") (net 1))
   (segment (start 107.338447 46.632447) (end 107.442 46.736) (width 0.3) (layer "F.Cu") (net 1))
@@
   (via (at 113.03 48.6664) (size 0.4572) (drill 0.254) (layers "F.Cu" "B.Cu") (free) (net 1))
   (via (at 103.378 57.7596) (size 0.4572) (drill 0.254) (layers "F.Cu" "B.Cu") (free) (net 1))
-  (via (at 105.156 49.3268) (size 0.4572) (drill 0.254) (layers "F.Cu" "B.Cu") (net 1))
   (via (at 104.648 41.656) (size 0.4572) (drill 0.254) (layers "F.Cu" "B.Cu") (free) (net 1))
   (via (at 101.7524 47.8536) (size 0.4572) (drill 0.254) (layers "F.Cu" "B.Cu") (free) (net 1))
@@
   (arc (start 110.660554 50.680246) (mid 110.76894 50.518034) (end 110.807 50.326693) (width 0.2) (layer "F.Cu") (net 11))
   (segment (start 104.267 53.594) (end 104.331 53.594) (width 0.2) (layer "F.Cu") (net 12))
-  (segment (start 103.651447 49.358153) (end 103.7844 49.2252) (width 0.2) (layer "F.Cu") (net 12))
-  (segment (start 103.739553 50.755153) (end 103.651446 50.667046) (width 0.2) (layer "F.Cu") (net 12))
-  (segment (start 104.542493 50.9016) (end 104.093107 50.9016) (width 0.2) (layer "F.Cu") (net 12))
-  (segment (start 103.505 50.313493) (end 103.505 49.711707) (width 0.2) (layer "F.Cu") (net 12))
+  (segment (start 105.156 50.507203) (end 105.156 49.381507) (width 0.2) (layer "F.Cu") (net 12))
   (segment (start 102.679 55.182) (end 104.267 53.594) (width 0.2) (layer "F.Cu") (net 12))
   (segment (start 102.679 55.372) (end 102.679 55.182) (width 0.2) (layer "F.Cu") (net 12))
-  (segment (start 104.9814 52.189893) (end 104.9814 51.1334) (width 0.2) (layer "F.Cu") (net 12))
-  (segment (start 104.9814 51.1334) (end 104.896046 51.048046) (width 0.2) (layer "F.Cu") (net 12))
-  (segment (start 104.642047 49.078753) (end 105.808054 47.912746) (width 0.2) (layer "F.Cu") (net 12))
-  (segment (start 104.477447 52.900953) (end 104.834954 52.543446) (width 0.2) (layer "F.Cu") (net 12))
-  (segment (start 105.9545 47.559193) (end 105.9545 47.486) (width 0.2) (layer "F.Cu") (net 12))
-  (segment (start 104.331 53.594) (end 104.331 53.254507) (width 0.2) (layer "F.Cu") (net 12))
-  (segment (start 103.7844 49.2252) (end 104.288493 49.2252) (width 0.2) (layer "F.Cu") (net 12))
-  (arc (start 103.651447 49.358153) (mid 103.54306 49.520365) (end 103.505 49.711707) (width 0.2) (layer "F.Cu") (net 12))
-  (arc (start 104.642047 49.078753) (mid 104.479835 49.18714) (end 104.288493 49.2252) (width 0.2) (layer "F.Cu") (net 12))
-  (arc (start 105.9545 47.559193) (mid 105.91644 47.750534) (end 105.808054 47.912746) (width 0.2) (layer "F.Cu") (net 12))
-  (arc (start 104.093107 50.9016) (mid 103.901765 50.86354) (end 103.739553 50.755153) (width 0.2) (layer "F.Cu") (net 12))
-  (arc (start 104.542493 50.9016) (mid 104.733834 50.93966) (end 104.896046 51.048046) (width 0.2) (layer "F.Cu") (net 12))
-  (arc (start 104.9814 52.189893) (mid 104.94334 52.381234) (end 104.834954 52.543446) (width 0.2) (layer "F.Cu") (net 12))
-  (arc (start 103.505 50.313493) (mid 103.54306 50.504834) (end 103.651446 50.667046) (width 0.2) (layer "F.Cu") (net 12))
-  (arc (start 104.477447 52.900953) (mid 104.36906 53.063165) (end 104.331 53.254507) (width 0.2) (layer "F.Cu") (net 12))
+  (segment (start 104.477447 53.002553) (end 104.834954 52.645046) (width 0.2) (layer "F.Cu") (net 12))
+  (segment (start 105.9545 48.168793) (end 105.9545 47.486) (width 0.2) (layer "F.Cu") (net 12))
+  (segment (start 104.9814 52.291493) (end 104.9814 50.88891) (width 0.2) (layer "F.Cu") (net 12))
+  (segment (start 104.9814 50.88891) (end 105.009554 50.860756) (width 0.2) (layer "F.Cu") (net 12))
+  (segment (start 104.331 53.594) (end 104.331 53.356107) (width 0.2) (layer "F.Cu") (net 12))
+  (segment (start 105.302447 49.027953) (end 105.808054 48.522346) (width 0.2) (layer "F.Cu") (net 12))
+  (arc (start 105.9545 48.168793) (mid 105.91644 48.360134) (end 105.808054 48.522346) (width 0.2) (layer "F.Cu") (net 12))
+  (arc (start 104.477447 53.002553) (mid 104.36906 53.164765) (end 104.331 53.356107) (width 0.2) (layer "F.Cu") (net 12))
+  (arc (start 104.834954 52.645046) (mid 104.94334 52.482834) (end 104.9814 52.291493) (width 0.2) (layer "F.Cu") (net 12))
+  (arc (start 105.156 49.381507) (mid 105.19406 49.190165) (end 105.302447 49.027953) (width 0.2) (layer "F.Cu") (net 12))
+  (arc (start 105.156 50.507203) (mid 105.11794 50.698544) (end 105.009554 50.860756) (width 0.2) (layer "F.Cu") (net 12))
   (segment (start 108.9295 45.986) (end 110.713393 45.986) (width 0.3) (layer "F.Cu") (net 13))
   (segment (start 111.066947 45.839553) (end 111.506 45.4005) (width 0.3) (layer "F.Cu") (net 13))
